File: PCB/hackCLUB.kicad_pcb (KiCad board)
At the start: 2 copper layers, 65.7 x 67.2 mm, 8 parts, among them SW1 SW_Push, SW2 SW_Push, SW3 SW_Push, SW4 SW_Push, SW5 RotaryEncoder_Switch, U1 XIAO-RP2040-DIP

Commit message: Changing the PCB
Routing:
- net +5V: track 35.7 -> 54.7 mm, vias 2 -> 0
- net GND: track 157.8 -> 166.2 mm, vias 0 -> 4
- net Net-(D1-DIN): track 10.2 -> 14.5 mm, vias 0 -> 1
- net Net-(D1-DOUT): track 21.0 -> 22.9 mm, vias 2 -> 0
Changed lines of the file:
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@@
+	)
+	(segment
+		(start 125.82 30.01)
+		(end 117.02 30.01)
+		(width 0.2)
+		(layer "F.Cu")
+		(net 1)
+	)
+	(segment
+		(start 115.723 34.027)
+		(end 104.413 34.027)
+		(width 0.2)
+		(layer "F.Cu")
+		(net 1)
+	)
+	(segment
+		(start 104.413 34.027)
+		(end 104.41 34.03)
+		(width 0.2)
+		(layer "F.Cu")
+		(net 1)
 	)
 	(segment
@@
 	)
 	(segment
-		(start 120.23 52.07)
-		(end 111.835 52.07)
-		(width 0.2)
-		(layer "F.Cu")
-		(net 1)
-	)
-	(segment
-		(start 99.775 31.015)
-		(end 98.09 32.7)
-		(width 0.2)
-		(layer "F.Cu")
-		(net 1)
-	)
-	(segment
-		(start 111.835 52.07)
-		(end 99.84 40.075)
+		(start 99.84 40.075)
+		(end 95.46 35.695)
+		(width 0.2)
+		(layer "F.Cu")
+		(net 1)
+	)
+	(segment
+		(start 116.9 32.85)
+		(end 115.723 34.027)
+		(width 0.2)
+		(layer "F.Cu")
+		(net 1)
+	)
+	(segment
+		(start 95.46 35.695)
+		(end 95.46 35.575)
+		(width 0.2)
+		(layer "F.Cu")
+		(net 1)
+	)
+	(segment
+		(start 100.76 33.44)
+		(end 100.76 33.39)
+		(width 0.2)
+		(layer "F.Cu")
+		(net 1)
+	)
+	(segment
+		(start 100.02 32.65)
+		(end 100.02 31.015)
 		(width 0.2)
 		(layer "F.Cu")
@@
 	)
 	(segment
-		(start 98.09 38.325)
-		(end 99.84 40.075)
-		(width 0.2)
-		(layer "F.Cu")
-		(net 1)
-	)
-	(segment
 		(start 100.02 31.015)
 		(end 99.775 31.015)
@@
 	)
 	(segment
+		(start 100.76 33.39)
+		(end 100.02 32.65)
+		(width 0.2)
+		(layer "F.Cu")
+		(net 1)
+	)
+	(segment
 		(start 120.23 71.14)
 		(end 120.27 71.18)
@@
 	)
 	(segment
-		(start 98.09 32.7)
-		(end 98.09 38.325)
-		(width 0.2)
-		(layer "F.Cu")
+		(start 117.02 30.01)
+		(end 116.94 29.93)
+		(width 0.2)
+		(layer "F.Cu")
+		(net 1)
+	)
+	(segment
+		(start 95.46 35.575)
+		(end 100.02 31.015)
+		(width 0.2)
+		(layer "F.Cu")
+		(net 1)
+	)
+	(via
+		(at 116.9 32.85)
+		(size 0.6)
+		(drill 0.3)
+		(layers "F.Cu" "B.Cu")
+		(net 1)
+	)
+	(via
+		(at 100.76 33.44)
+		(size 0.6)
+		(drill 0.3)
+		(layers "F.Cu" "B.Cu")
+		(net 1)
+	)
+	(via
+		(at 116.94 29.93)
+		(size 0.6)
+		(drill 0.3)
+		(layers "F.Cu" "B.Cu")
+		(net 1)
+	)
+	(via
+		(at 104.41 34.03)
+		(size 0.6)
+		(drill 0.3)
+		(layers "F.Cu" "B.Cu")
 		(net 1)
 	)
@@
 	)
 	(segment
+		(start 116.94 32.81)
+		(end 116.9 32.85)
+		(width 0.2)
+		(layer "B.Cu")
+		(net 1)
+	)
+	(segment
+		(start 116.94 29.93)
+		(end 116.94 32.81)
+		(width 0.2)
+		(layer "B.Cu")
+		(net 1)
+	)
+	(segment
 		(start 120.23 52.07)
 		(end 130.119 42.181)
@@
 	)
 	(segment
+		(start 103.82 33.44)
+		(end 100.76 33.44)
+		(width 0.2)
+		(layer "B.Cu")
+		(net 1)
+	)
+	(segment
 		(start 125.82 30.09)
 		(end 125.82 30.01)
@@
 	)
 	(segment
-		(start 103.52 29.265)
-		(end 106.685 26.1)
-		(width 0.2)
-		(layer "F.Cu")
-		(net 2)
-	)
-	(segment
-		(start 103.34 38.325)
-		(end 103.34 36.17)
-		(width 0.2)
-		(layer "F.Cu")
-		(net 2)
-	)
-	(segment
-		(start 104.575 30.32)
+		(start 104.41 34.03)
+		(end 103.82 33.44)
+		(width 0.2)
+		(layer "B.Cu")
+		(net 1)
+	)
+	(segment
+		(start 103.34 33.3029)
+		(end 103.34 38.325)
+		(width 0.2)
+		(layer "F.Cu")
+		(net 2)
+	)
+	(segment
+		(start 125.82 27.47)
+		(end 124.757 26.407)
+		(width 0.2)
+		(layer "F.Cu")
+		(net 2)
+	)
+	(segment
+		(start 106.378 26.407)
 		(end 103.52 29.265)
 		(width 0.2)
@@
 	)
 	(segment
-		(start 124.45 26.1)
-		(end 125.82 27.47)
-		(width 0.2)
-		(layer "F.Cu")
-		(net 2)
-	)
-	(segment
-		(start 105.68 30.32)
-		(end 104.575 30.32)
-		(width 0.2)
-		(layer "F.Cu")
-		(net 2)
-	)
-	(segment
-		(start 106.685 26.1)
-		(end 124.45 26.1)
-		(width 0.2)
-		(layer "F.Cu")
-		(net 2)
-	)
-	(segment
-		(start 103.34 36.17)
-		(end 105.19 34.32)
-		(width 0.2)
-		(layer "F.Cu")
-		(net 2)
-	)
-	(via
-		(at 105.19 34.32)
-		(size 0.6)
-		(drill 0.3)
-		(layers "F.Cu" "B.Cu")
-		(net 2)
-	)
-	(via
-		(at 105.68 30.32)
-		(size 0.6)
-		(drill 0.3)
-		(layers "F.Cu" "B.Cu")
-		(net 2)
-	)
-	(segment
-		(start 105.68 33.83)
-		(end 105.68 30.32)
-		(width 0.2)
-		(layer "B.Cu")
-		(net 2)
-	)
-	(segment
-		(start 105.19 34.32)
-		(end 105.68 33.83)
-		(width 0.2)
-		(layer "B.Cu")
-		(net 2)
-	)
-	(segment
-		(start 103.52 31.64)
-		(end 109.51 37.63)
-		(width 0.2)
-		(layer "F.Cu")
-		(net 3)
+		(start 108.0969 28.546)
+		(end 103.34 33.3029)
+		(width 0.2)
+		(layer "F.Cu")
+		(net 2)
+	)
+	(segment
+		(start 124.757 26.407)
+		(end 106.378 26.407)
+		(width 0.2)
+		(layer "F.Cu")
+		(net 2)
+	)
+	(segment
+		(start 126.655 27.47)
+		(end 125.579 28.546)
+		(width 0.2)
+		(layer "F.Cu")
+		(net 2)
+	)
+	(segment
+		(start 125.579 28.546)
+		(end 108.0969 28.546)
+		(width 0.2)
+		(layer "F.Cu")
+		(net 2)
 	)
 	(segment
@@
 	)
 	(segment
+		(start 104.955 29.58)
+		(end 105.56 29.58)
+		(width 0.2)
+		(layer "F.Cu")
+		(net 3)
+	)
+	(segment
 		(start 103.52 31.015)
 		(end 103.52 31.64)
@@
 	)
 	(segment
-		(start 97.25 29.62)
-		(end 97.605 29.265)
-		(width 0.2)
-		(layer "F.Cu")
-		(net 4)
-	)
-	(segment
-		(start 105.01 38.405)
-		(end 105.01 35.92)
-		(width 0.2)
-		(layer "F.Cu")
-		(net 4)
-	)
-	(segment
-		(start 97.605 29.265)
-		(end 100.02 29.265)
-		(width 0.2)
-		(layer "F.Cu")
-		(net 4)
-	)
-	(segment
-		(start 103.34 40.075)
-		(end 105.01 38.405)
-		(width 0.2)
-		(layer "F.Cu")
-		(net 4)
-	)
-	(via
-		(at 97.25 29.62)
-		(size 0.6)
-		(drill 0.3)
-		(layers "F.Cu" "B.Cu")
-		(net 4)
-	)
-	(via
-		(at 105.01 35.92)
-		(size 0.6)
-		(drill 0.3)
-		(layers "F.Cu" "B.Cu")
-		(net 4)
-	)
-	(segment
-		(start 104.85 35.76)
-		(end 99.08 35.76)
-		(width 0.2)
-		(layer "B.Cu")
-		(net 4)
-	)
-	(segment
-		(start 105.01 35.92)
-		(end 104.85 35.76)
-		(width 0.2)
-		(layer "B.Cu")
-		(net 4)
-	)
-	(segment
-		(start 97.22 29.65)
-		(end 97.25 29.62)
-		(width 0.2)
-		(layer "B.Cu")
-		(net 4)
-	)
-	(segment
-		(start 99.08 35.76)
-		(end 98.53 35.76)
-		(width 0.2)
-		(layer "B.Cu")
-		(net 4)
-	)
-	(segment
-		(start 97.22 34.45)
-		(end 97.22 29.65)
-		(width 0.2)
-		(layer "B.Cu")
-		(net 4)
-	)
-	(segment
-		(start 98.53 35.76)
-		(end 97.22 34.45)
-		(width 0.2)
-		(layer "B.Cu")
-		(net 4)
-	)
+		(start 103.52 31.015)
+		(end 104.955 29.58)
+		(width 0.2)
+		(layer "F.Cu")
+		(net 3)
+	)
+	(via
+		(at 105.56 29.58)
+		(size 0.6)
+		(drill 0.3)
+		(layers "F.Cu" "B.Cu")
+		(net 3)
+	)
+	(segment
+		(start 105.56 32.61)
+		(end 110.58 37.63)
+		(width 0.2)
+		(layer "B.Cu")
+		(net 3)
+	)
+	(segment
+		(start 105.56 29.58)
+		(end 105.56 32.61)
+		(width 0.2)
+		(layer "B.Cu")
+		(net 3)
+	)
+	(segment
+		(start 101.035 42.38)
+		(end 103.34 40.075)
+		(width 0.2)
+		(layer "F.Cu")
+		(net 4)
+	)
+	(segment
+		(start 99.93 42.38)
+		(end 101.035 42.38)
+		(width 0.2)
+		(layer "F.Cu")
+		(net 4)
+	)
+	(segment
+		(start 99.985 29.265)
+		(end 93.4 35.85)
+		(width 0.2)
+		(layer "F.Cu")
+		(net 4)
+	)
+	(segment
+		(start 93.4 35.85)
+		(end 99.93 42.38)
+		(width 0.2)
+		(layer "F.Cu")
+		(net 4)
+	)
+	(segment
+		(start 100.02 29.265)
+		(end 99.985 29.265)
+		(width 0.2)
+		(layer "F.Cu")
+		(net 4)
+	)
